Commit message: Checkpoint ASV PPO training fixes

File: yf_description/urdf/base_asv.xacro (robot description, xacro)
@@ -4,11 +4,10 @@
     <link
       name="${name}/base_link">
-      <visual>
+      <visual name="hull">
         <origin
           xyz="0 0 0"
-          rpy="0 0 ${pi/2}" />
+          rpy="0 0 0" />
         <geometry>
-          <mesh
-            filename="package://yf_description/meshes/base_link.STL" />
+          <box size="0.95 0.48 0.16" />
         </geometry>
         <material
@@ -54,8 +53,7 @@
         <origin
           xyz="0 0 0"
-          rpy="0 0 ${pi/2}" />
+          rpy="0 0 0" />
         <geometry>
-          <mesh
-            filename="package://yf_description/meshes/base_link.STL" />
+          <box size="0.95 0.48 0.16" />
         </geometry>
       </collision>
@@ -68,6 +66,5 @@
           rpy="0 0 0" />
         <geometry>
-          <mesh
-            filename="package://yf_description/meshes/Motor_izquierda_link.STL" />
+          <box size="0.18 0.08 0.08" />
         </geometry>
         <material
@@ -82,6 +79,5 @@
           rpy="0 0 0" />
         <geometry>
-          <mesh
-            filename="package://yf_description/meshes/Motor_izquierda_link.STL" />
+          <box size="0.18 0.08 0.08" />
         </geometry>
       </collision>
@@ -94,6 +90,5 @@
           rpy="0 0 0" />
         <geometry>
-          <mesh
-            filename="package://yf_description/meshes/Motor_derecha_link.STL" />
+          <box size="0.18 0.08 0.08" />
         </geometry>
         <material
@@ -108,6 +103,5 @@
           rpy="0 0 0" />
         <geometry>
-          <mesh
-            filename="package://yf_description/meshes/Motor_derecha_link.STL" />
+          <box size="0.18 0.08 0.08" />
         </geometry>
       </collision>

File: yf_description/urdf/base_neighbor.xacro (robot description, xacro)
@@ -4,11 +4,10 @@
     <link
       name="${name}/base_link">
-      <visual>
+      <visual name="hull">
         <origin
           xyz="0 0 0"
-          rpy="0 0 ${pi/2}" />
+          rpy="0 0 0" />
         <geometry>
-          <mesh
-            filename="package://yf_description/meshes/base_link.STL" />
+          <box size="0.95 0.48 0.16" />
         </geometry>
         <material
@@ -54,8 +53,7 @@
         <origin
           xyz="0 0 0"
-          rpy="0 0 ${pi/2}" />
+          rpy="0 0 0" />
         <geometry>
-          <mesh
-            filename="package://yf_description/meshes/base_link.STL" />
+          <box size="0.95 0.48 0.16" />
         </geometry>
       </collision>
@@ -68,6 +66,5 @@
           rpy="0 0 0" />
         <geometry>
-          <mesh
-            filename="package://yf_description/meshes/Motor_izquierda_link.STL" />
+          <box size="0.18 0.08 0.08" />
         </geometry>
         <material
@@ -82,6 +79,5 @@
           rpy="0 0 0" />
         <geometry>
-          <mesh
-            filename="package://yf_description/meshes/Motor_izquierda_link.STL" />
+          <box size="0.18 0.08 0.08" />
         </geometry>
       </collision>
@@ -94,6 +90,5 @@
           rpy="0 0 0" />
         <geometry>
-          <mesh
-            filename="package://yf_description/meshes/Motor_derecha_link.STL" />
+          <box size="0.18 0.08 0.08" />
         </geometry>
         <material
@@ -108,6 +103,5 @@
           rpy="0 0 0" />
         <geometry>
-          <mesh
-            filename="package://yf_description/meshes/Motor_derecha_link.STL" />
+          <box size="0.18 0.08 0.08" />
         </geometry>
       </collision>

File: yf_description/urdf/components/asv_gps.xacro (robot description, xacro)
@@ -22,10 +22,10 @@
     <joint name="${name}/gps_joint" type="fixed">
       <origin
-        xyz="0.27 0.28 -0.54"
+        xyz="-0.27 -0.28 0.54"
         rpy="0 0 0" />
       <parent
+        link="${name}/base_link" />
+      <child
         link="${name}/gps_link" />
-      <child
-        link="${name}/base_link" />
     </joint>
   </xacro:macro>
